File: powm.kicad_sch (KiCad schematic)
At the start: 9 parts, among them J1 USB_C_Receptacle_PowerOnly_6P, U1 IP2721, U2 BQ25792RQMR

Commit message: 1
Parts:
- removed TP1: USB V+, TestPoint:TestPoint_Pad_D1.0mm, symbol Connector:TestPoint
- added Q1: PMOS, symbol Simulation_SPICE:PMOS
- added Q2: IRLR2905, Package_TO_SOT_SMD:TO-252-2, symbol Simulation_SPICE:NMOS
- added R4: 500, Resistor_SMD:R_0603_1608Metric_Pad0.98x0.95mm_HandSolder, symbol Device:R
- added R5: 100k, Resistor_SMD:R_0603_1608Metric_Pad0.98x0.95mm_HandSolder, symbol Device:R
- added TP2: USB V+, TestPoint:TestPoint_Pad_1.0x1.0mm, symbol Connector:TestPoint
- C2: value 1uF -> 10uF
- U2: footprint Library:QFN40P400X400X100-29N -> Package_DFN_QFN:Texas_RQM0029A_VQFN-29_4x4mm_P0.4mm
Connections:
- net GND: now also R5.2
- net VAC1: now also Q2.3 (S)
- net at C1.1, J1.A9 (VBUS), J1.B9 (VBUS)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: now also Q2.1 (D), TP2.1
- net at U1.1 (VBUSG): now also R4.2
- new net: Q2.2 (G), R4.1, R5.1
Other:
- moved on the sheet: C2, U2
