File: powm.kicad_sch (KiCad schematic)
At the start: 13 parts, among them J1 USB_C_Receptacle_PowerOnly_6P, Q1 PMOS, Q2 IRLR2905, U1 IP2721, U2 BQ25792RQMR

Commit message: add sym lib
Parts:
- removed U2: BQ25792RQMR, Package_DFN_QFN:Texas_RQM0029A_VQFN-29_4x4mm_P0.4mm, symbol BQ25792RQMR:BQ25792RQMR
- added U3: BQ25792, Package_DFN_QFN:Texas_RQM0029A_VQFN-29_4x4mm_P0.4mm, symbol powm:BQ25792
Changed lines of the file:
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@@
-	(wire
-		(pts
-			(xy 297.18 74.93) (xy 307.34 74.93)
-		)
-		(stroke
-			(width 0)
-			(type default)
-		)
-	)
 	(wire
 		(pts
@@
 				(thickness 0.254)
 				(bold yes)
-			)
-			(justify left bottom)
-		)
-	)
-	(label "VAC1"
-		(at 297.18 74.93 0)
-		(effects
-			(font
-				(size 1.27 1.27)
 			)
 			(justify left bottom)
@@
 	)
 	(symbol
-		(lib_id "BQ25792RQMR:BQ25792RQMR")
-		(at 327.66 77.47 0)
-		(unit 1)
-		(exclude_from_sim no)
-		(in_bom yes)
-		(on_board yes)
-		(dnp no)
-		(fields_autoplaced yes)
-		(property "Reference" "U2"
-			(at 327.66 39.37 0)
-			(effects
-				(font
-					(size 1.27 1.27)
-				)
-			)
-		)
-		(property "Value" "BQ25792RQMR"
-			(at 327.66 41.91 0)
-			(effects
-				(font
-					(size 1.27 1.27)
-				)
-			)
-		)
-		(property "Footprint" "Package_DFN_QFN:Texas_RQM0029A_VQFN-29_4x4mm_P0.4mm"
-			(at 327.66 77.47 0)
-			(effects
-				(font
-					(size 1.27 1.27)
-				)
-				(justify bottom)
-				(hide yes)
-			)
-		)
-		(property "Datasheet" "Datasheets/bq25792.pdf"
-			(at 327.66 77.47 0)
-			(effects
-				(font
-					(size 1.27 1.27)
-				)
-				(hide yes)
-			)
-		)
-		(property "Description" ""
-			(at 327.66 77.47 0)
-			(effects
-				(font
-					(size 1.27 1.27)
-				)
-				(hide yes)
-			)
-		)
-		(property "PARTREV" "11/2019"
-			(at 327.66 77.47 0)
-			(effects
-				(font
-					(size 1.27 1.27)
-				)
-				(justify bottom)
-				(hide yes)
-			)
-		)
-		(property "STANDARD" "Manufacturer Recommendations"
-			(at 327.66 77.47 0)
-			(effects
-				(font
-					(size 1.27 1.27)
-				)
-				(justify bottom)
-				(hide yes)
-			)
-		)
-		(property "MAXIMUM_PACKAGE_HEIGHT" "1 mm"
-			(at 327.66 77.47 0)
-			(effects
-				(font
-					(size 1.27 1.27)
-				)
-				(justify bottom)
-				(hide yes)
-			)
-		)
-		(property "MANUFACTURER" "Texas Instruments"
-			(at 327.66 77.47 0)
-			(effects
-				(font
-					(size 1.27 1.27)
-				)
-				(justify bottom)
-				(hide yes)
-			)
-		)
-		(pin "1"
-		)
-		(pin "10"
-		)
-		(pin "11"
-		)
-		(pin "12"
-		)
-		(pin "13"
-		)
-		(pin "14"
-		)
-		(pin "15"
-		)
-		(pin "16"
-		)
-		(pin "17"
-		)
-		(pin "18"
-		)
-		(pin "19"
-		)
-		(pin "2"
-		)
-		(pin "20"
-		)
-		(pin "21"
-		)
-		(pin "22"
-		)
-		(pin "23"
-		)
-		(pin "24"
-		)
-		(pin "25"
-		)
-		(pin "26"
-		)
-		(pin "27"
-		)
-		(pin "28"
-		)
-		(pin "29"
-		)
-		(pin "3"
-		)
-		(pin "4"
-		)
-		(pin "5"
-		)
-		(pin "6"
-		)
-		(pin "7"
-		)
-		(pin "8"
-		)
-		(pin "9"
-		)
-		(instances
-			(project "powm"
-				(path "/b8a951bd-38c7-4b6e-9d63-c1fe34e675e5"
-					(reference "U2")
-					(unit 1)
-				)
-			)
-		)
-	)
-	(symbol
 		(lib_id "Simulation_SPICE:NMOS")
 		(at 119.38 36.83 90)
@@
 					(unit 1)
 				)
+			)
+		)
+	)
+	(symbol
+		(lib_id "powm:BQ25792")
+		(at 240.03 63.5 0)
+		(unit 1)
+		(exclude_from_sim no)
+		(in_bom yes)
+		(on_board yes)
+		(dnp no)
+		(fields_autoplaced yes)
+		(property "Reference" "U3"
+			(at 240.03 35.56 0)
+			(effects
+				(font
+					(size 1.27 1.27)
+				)
+			)
+		)
+		(property "Value" "BQ25792"
+			(at 240.03 38.1 0)
+			(effects
+				(font
+					(size 1.27 1.27)
+				)
+			)
+		)
+		(property "Footprint" "Package_DFN_QFN:Texas_RQM0029A_VQFN-29_4x4mm_P0.4mm"
+			(at 240.03 63.5 0)
+			(effects
+				(font
+					(size 1.27 1.27)
+				)
+				(hide yes)
+			)
+		)
+		(property "Datasheet" ""
+			(at 240.03 63.5 0)
+			(effects
+				(font
+					(size 1.27 1.27)
+				)
+				(hide yes)
+			)
+		)
+		(property "Description" ""
+			(at 240.03 63.5 0)
+			(effects
+				(font
+					(size 1.27 1.27)
+				)
+				(hide yes)
+			)
+		)
+		(pin "11"
+		)
+		(pin "13"
+		)
+		(pin "1"
+		)
+		(pin "24"
+		)
+		(pin "6"
+		)
+		(pin "20"
+		)
+		(pin "4"
+		)
+		(pin "16"
+		)
+		(pin "3"
+		)
+		(pin "9"
+		)
+		(pin "10"
+		)
+		(pin "12"
+		)
+		(pin "14"
+		)
+		(pin "26"
+		)
+		(pin "15"
+		)
+		(pin "7"
+		)
+		(pin "2"
+		)
+		(pin "29"
+		)
+		(pin "27"
+		)
+		(pin "25"
+		)
+		(pin "8"
+		)
+		(pin "5"
+		)
+		(pin "28"
+		)
+		(pin "23"
+		)
+		(pin "22"
+		)
+		(pin "21"
+		)
+		(pin "19"
+		)
+		(pin "18"
+		)
+		(pin "17"
+		)
+		(instances
+			(project ""
+				(path "/b8a951bd-38c7-4b6e-9d63-c1fe34e675e5"
+					(reference "U3")
+					(unit 1)
+				)

Commit message: 2
Parts:
- removed Q1: PMOS, symbol Simulation_SPICE:PMOS
- added C10, C11, C13, C14, C15, C16, C6, C7, C9: 10uF, Capacitor_SMD:C_0603_1608Metric_Pad1.08x0.95mm_HandSolder, symbol Device:C
- added C12, C3, C4, C5, C8: 0.1uF, Capacitor_SMD:C_0603_1608Metric_Pad1.08x0.95mm_HandSolder, symbol Device:C
- added D1, D2: BZT52C12T-7, Diode_SMD:D_SOD-523, symbol Device:D_Zener
- added Q1, Q3, Q4, Q5: IRLR2905, Package_TO_SOT_SMD:TO-252-2, symbol Simulation_SPICE:NMOS
- added R6, R7: 250, Resistor_SMD:R_0603_1608Metric_Pad0.98x0.95mm_HandSolder, symbol Device:R
- added TP1: VAC2, TestPoint:TestPoint_THTPad_D4.0mm_Drill2.0mm, symbol Connector:TestPoint
Connections:
- net GND: now also C10.2, C11.2, C12.2, C13.2, C14.2, C15.2, C16.2, C3.2, C4.2, C5.2, C6.2, C7.2, C8.2, C9.2
- net VAC1: now also U3.9 (VAC1), C3.1, Q4.1 (D)
- net ACDRV2: now reaches U3.10 (ACDRV2)
- net ACDRV2: now also R6.2
- net ACDRV1: now reaches U3.11 (ACDRV1)
- net ACDRV1: now also R7.2
- net VBUS: now reaches U3.2 (VBUS)
- net VBUS: now also U3.3 (VBUS), C5.1, C6.1, C7.1, Q3.1 (D), Q5.1 (D)
- net SYS: now reaches U3.25 (SYS)
- net SYS: now also C12.1, C13.1, C14.1, C15.1, C16.1
- net PMID: now reaches U3.29 (PMID)
- net PMID: now also C10.1, C11.1, C8.1, C9.1
- net VAC2: now reaches U3.8 (VAC2)
- net VAC2: now also C4.1, Q1.1 (D), TP1.1
- new net: D2.1 (K), Q1.2 (G), Q3.2 (G), R6.1
- new net: D2.2 (A), Q1.3 (S), Q3.3 (S)
- new net: D1.1 (K), Q4.2 (G), Q5.2 (G), R7.1
- new net: D1.2 (A), Q4.3 (S), Q5.3 (S)
Other:
- moved on the sheet: U3

Commit message: 4
Parts:
- added C17, C18: 47uF, Capacitor_SMD:C_0603_1608Metric_Pad1.08x0.95mm_HandSolder, symbol Device:C
- added C19: 4.7uF, Capacitor_SMD:C_0603_1608Metric_Pad1.08x0.95mm_HandSolder, symbol Device:C
- added C20: 1nF, Capacitor_SMD:C_0603_1608Metric_Pad1.08x0.95mm_HandSolder, symbol Device:C
- added C21, C22: 10uF, Capacitor_SMD:C_0603_1608Metric_Pad1.08x0.95mm_HandSolder, symbol Device:C
- added D3: LED, symbol Device:LED
- added L1: 2.2uH, symbol Device:L
- added R10: 5.24k, Resistor_SMD:R_0603_1608Metric_Pad0.98x0.95mm_HandSolder, symbol Device:R
- added R11: 100k, Resistor_SMD:R_0603_1608Metric_Pad0.98x0.95mm_HandSolder, symbol Device:R
- added R12: 127k, Resistor_SMD:R_0603_1608Metric_Pad0.98x0.95mm_HandSolder, symbol Device:R
- added R13: 27k, Resistor_SMD:R_0603_1608Metric_Pad0.98x0.95mm_HandSolder, symbol Device:R
- added R14: 100, Resistor_SMD:R_0603_1608Metric_Pad0.98x0.95mm_HandSolder, symbol Device:R
- added R8: 2.2k, Resistor_SMD:R_0603_1608Metric_Pad0.98x0.95mm_HandSolder, symbol Device:R
- added R9: 30.31k, Resistor_SMD:R_0603_1608Metric_Pad0.98x0.95mm_HandSolder, symbol Device:R
- added TP3: TH, TestPoint:TestPoint_THTPad_D2.0mm_Drill1.0mm, symbol Connector:TestPoint
- added TP4: TH_GND, TestPoint:TestPoint_THTPad_D2.0mm_Drill1.0mm, symbol Connector:TestPoint
- added TP5: BAT+, TestPoint:TestPoint_THTPad_D2.0mm_Drill1.0mm, symbol Connector:TestPoint
- added TP6: BAT-, TestPoint:TestPoint_THTPad_D2.0mm_Drill1.0mm, symbol Connector:TestPoint
Connections:
- net GND: now also U3.13 (CE), U3.27 (GND), C19.2, C20.2, C21.2, C22.2, R10.1, R11.1, R13.2, TP4.1, TP6.1
- net at U3.1 (STAT): now also D3.1 (K)
- net I2C_SCL: now reaches U3.14 (SCL)
- net I2C_SDA: now reaches U3.15 (SDA)
- net at U3.16 (TS): now also R10.2, R9.1, TP3.1
- net at U3.17 (ILIM_HIZ): now also R11.2, R12.1
- net BATP: now reaches U3.18 (BATP)
- net BATP: now also R14.1
- net BTST2: now reaches U3.19 (BTST2)
- net BTST2: now also C18.2
- net at U3.20 (PROG): now also R13.1
- net BAT: now reaches U3.22 (BAT)
- net BAT: now also U3.23 (BAT), C21.1, C22.1, R14.2, TP5.1
- net SDRV: now reaches U3.24 (SDRV)
- net SDRV: now also C20.1
- net at U3.26 (SW2): now also C18.1, L1.2
- net at U3.28 (SW1): now also C17.2, L1.1
- net BTST1: now reaches U3.4 (BTST1)
- net BTST1: now also C17.1
- net REGN: now reaches U3.5 (REGN)
- net REGN: now also C19.1, R12.2, R8.1, R9.2
- new net: D3.2 (A), R8.2
- no-connect marks 0 -> 3
Other:
- note added: "P/S 0.1мкФ как можно ближе к целевым выходам МК у каждого массива кап"
- moved on the sheet: C10, C11, C12, C13, C14, C15, C16, C5, C6, C7, C8, C9

Commit message: 1
Parts:
- added C23: 2.2uF, Capacitor_SMD:C_0603_1608Metric_Pad1.08x0.95mm_HandSolder, symbol Device:C
- added C24: 10uF, Capacitor_SMD:C_0603_1608Metric_Pad1.08x0.95mm_HandSolder, symbol Device:C
- added C25, C26: 1nF, Capacitor_SMD:C_0603_1608Metric_Pad1.08x0.95mm_HandSolder, symbol Device:C
- added D4, D5: SMBJ24CA, symbol Device:D_TVS
- added R15: 2, Resistor_SMD:R_0603_1608Metric_Pad0.98x0.95mm_HandSolder, symbol Device:R
- added TP7: VBUS, TestPoint:TestPoint_Pad_D1.0mm, symbol Connector:TestPoint
- added TP8: GND, TestPoint:TestPoint_THTPad_D4.0mm_Drill2.0mm, symbol Connector:TestPoint
- added TP9: SYS, TestPoint:TestPoint_Pad_D1.0mm, symbol Connector:TestPoint
- added U2: tps611781, symbol powm:tps611781
Connections:
- net BAT: now also D4.2 (A2)
- net GND: now also R9.1, C23.2, C24.2, D4.1 (A1), D5.1 (A1), TP8.1; no longer R10.1
- net REGN: now also R10.2; no longer R9.2
- net SYS: now also C24.1, TP9.1
- net VBUS: now also D5.2 (A2), R15.1, TP7.1
- net at D2.1 (K), Q1.2 (G), Q3.2 (G)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: now also C25.2
- net at D2.2 (A), Q1.3 (S), Q3.3 (S): now also C25.1
- net at D1.1 (K), Q4.2 (G), Q5.2 (G)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: now also C26.1
- net at TP3.1, U3.16 (TS): now also R10.1, R9.2; no longer R10.2, R9.1
- net at D1.2 (A), Q4.3 (S), Q5.3 (S): now also C26.2
- new net: C23.1, R15.2
- no-connect marks 3 -> 4
Other:
- note added: "103AT-2"
- moved on the sheet: C3, Q1, Q4, R10, R9
